File: fan-controller/fan-controller.kicad_sch (KiCad schematic)
At the start: 23 parts, among them J1 DC_Jack_12V, J2 FAN1, J3 FAN2, J4 FAN3, J5 FAN4, U1 XIAO ESP32-C3, U2 AMS1117-5.0

Commit message: Fold every schematic step into generate.py; swap fan pin pairs
generate.py is now the only command needed to rebuild the schematic. It runs
the full sequence, because each step used to be separate and every one of them
was forgotten at least once:

  1. reposition symbols and redraw all nets   (validated before writing)
  2. repair structural defects                (was fix_sch.py, now deleted)
  3. re-attach PWR_FLAGs and no-connects      (was an ad-hoc snippet, retyped
                                               by hand three times)
  4. verify the netlist against netplan.py    (was a separate audit)

Step 4 matters most: ERC cannot catch a wire landing on the wrong real pin,
since that is still a legal connection. Only a pin-by-pin netlist diff does.
--no-verify skips it where kicad-cli is unavailable.

Two latent bugs fixed while integrating:

  * Placed symbols were matched with a single-line regex, but KiCad rewrites
    the file with each field on its own line whenever the schematic is opened
    in the GUI. Regenerating after any GUI session found zero symbols and
    failed; fix_sch.py hit the same thing but failed silently, reporting
    success while repairing nothing. Both paths now use a whitespace-tolerant
    SYMBOL_RE, and a symbol's (at ...) is rewritten by matched span rather
    than by reconstructing the literal text.

  * netplan.py had lost pin_abs_rot, which only ever existed in a session
    scratchpad that a crash wiped. Restored and re-verified empirically
    against all four rotations before use.

Also swaps the XIAO pins between FAN1/FAN2 and FAN3/FAN4 as requested:
  FAN1 D1/D2 (2,3)   FAN2 D3/D4 (4,5)
  FAN3 D7/D10 (8,11) FAN4 D5/D6 (6,7)

PCB synced: 16 U1 pad assignments updated (8 pins x 2, since the DIP
footprint pairs an SMD and a through-hole pad per number). All 22 nets
cross-checked between schematic and board.

Board also reworked earlier in this session: outline fitted to the ground
zone at 76.5 x 29 mm (was 80 x 60), J1 m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
Connections:
- net FAN3_PWM: now also U1.8 (D7); no longer U1.6 (D5)
- net FAN3_TACH: now also U1.11 (D10); no longer U1.7 (D6)
- net FAN4_PWM: now also U1.6 (D5); no longer U1.8 (D7)
- net FAN4_TACH: now also U1.7 (D6); no longer U1.11 (D10)

Commit message: Route the board: ground plane, wider power nets, jack on the edge
The PCB is now fully routed. 167 tracks, 7 vias, no unconnected pads.

Layout
  Board shrunk from 80 x 60 mm to 72.9 x 25.0 mm, fitted 1mm clear of all
  copper. J1 sits on the right end opposite the XIAO with its flange on the
  board edge, so the 3.5mm barrel protrudes as a panel-mount jack should.
  Getting there took two goes: the flange initially sat 1.9mm inboard of the
  edge, making the plug look adrift. Moving the plug pocket (J1, F1, D1 plus
  9 tracks) 1.8mm inward fixed it. 3mm was requested but drives F1's pad and
  the +12V_IN wire into the +12V_PROT trunk at x=91.5; 1.8mm is the limit
  before that clash. Only the 2 tracks crossing the pocket boundary needed
  shortening, exactly as predicted.

Ground plane
  GND pour on B.Cu, 1417mm^2, thermal relief on pads. A keep-out clears the
  copper away from the XIAO's antenna: U1 is rotated -90 so pins 7 and 8 both
  sit at y=59.88, the module's top edge, which is the antenna end opposite
  the USB connector. The window stops at y=58.6, clearing those two pads by
  0.52mm - an earlier attempt ran to y=60.0 and DRC rightly rejected it for
  swallowing them.

Track widths
  Power and ground widened from the 0.2mm minimum (0.74A) to targets from
  IPC-2152 at 1oz, 10C rise. A single width does not fit: the corridor around
  U1 is a 2.54mm pad pitch. So each segment starts at target and steps down
  only where DRC objects.

    +12V_IN, +12V_FUSED, +12V_PROT   1.0mm    2.39 A
    GND                              1.0mm    2.39 A  (2 segments 0.2mm)
    +5V, +3V3                        0.6mm    1.65 A

  The 12V rail feeds four fans through a 1.5A-hold polyfuse, so 2.39A leaves
  real margin. The two 0.2mm GND segments run directly over the B.Cu plane -
  sampling along their length found plane copper at 28 of 33 points, and U1's
  GND pad is a through-hole tied into it - so the plane carries that return
  in parallel and width is not the limit ther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
Connections:
- net FAN4_PWM: now also U1.7 (D6); no longer U1.6 (D5)
- net FAN4_TACH: now also U1.6 (D5); no longer U1.7 (D6)
Changed lines of the file:
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@@
 	(wire
 		(pts
-			(xy 33.41 126.43) (xy 30.87 126.43)
+			(xy 33.41 130.24) (xy 30.87 130.24)
 		)
 		(stroke
@@
 	)
 	(label "FAN4_PWM"
-		(at 30.87 126.43 180)
+		(at 30.87 130.24 180)
 		(effects
 			(font
@@
 	(wire
 		(pts
-			(xy 33.41 130.24) (xy 30.87 130.24)
+			(xy 33.41 126.43) (xy 30.87 126.43)
 		)
 		(stroke
@@
 	)
 	(label "FAN4_TACH"
-		(at 30.87 130.24 180)
+		(at 30.87 126.43 180)
 		(effects
 			(font

Commit message: Generate the fabrication package
make_fab.sh produces everything a fab house needs, in one command:
gerbers, Excellon drill, BOM and pick-and-place, zipped as
fab/fan-controller-fab.zip (15 files, 194 KB).

Board: 72.9 x 25.0 mm, 2 layers, min track/clearance 0.2mm, min drill
0.3mm, 42 holes across 5 sizes. Quantity 20, assembled.

Three things needed handling that the default exports get wrong:

  Gerbers must name their layers explicitly. A bare `kicad-cli pcb export
  gerbers` writes every layer - the first run shipped a 152KB User_Eco1.gbr
  containing the review markers used during layout.

  The four fan headers would not group in the BOM. Their Values are
  FAN1..FAN4 (which channel each drives), and kicad-cli's grouping compares
  every field, so one identical part appeared as four line items - an
  assembler would source four different connectors. make_bom.py regroups on
  footprint + part type and keeps the channel names in a Note column.

  The socket headers were missing entirely. U1 is socketed, so the 2x 1x7
  female headers are what actually gets assembled, but they have no
  schematic symbol - the XIAO's footprint provides their pads. Without an
  explicit BOM line they would simply not be fitted. Added, with the pad
  geometry confirmed from the board: 14 through-hole pads in two columns of
  7 at 2.54mm pitch.

U1 is now marked DNP in both schematic and board (the flag does not
propagate on its own without an Update-PCB-from-Schematic pass), so
--exclude-dnp drops it from the CPL: 22 placements, all top side.

Placement and drill files share an origin at the board's bottom-left
corner; there was no aux origin set, so --use-drill-file-origin had been
falling back to absolute coordinates with negative Y.

Verified: outline in the gerber measures 72.9 x 25.0mm, both copper layers
carry the expected geometry (B.Cu has filled regions for the ground pour),
zip integrity OK. ERC and DRC unchanged - no electrical errors.

fab/gerbers/ and the zip are gitig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
Parts:
- U1: now not fitted
Changed lines of the file:
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@@
 			)
 		)
-		(property "Description" ""
+		(property "Description" "4-pin fan header 2.54mm"
 			(at 168.0 84.0 0)
 			(show_name no)
@@
 			)
 		)
-		(property "Description" ""
+		(property "Description" "4-pin fan header 2.54mm"
 			(at 168.0 198.0 0)
 			(show_name no)
@@
 			)
 		)
-		(property "Description" ""
+		(property "Description" "4-pin fan header 2.54mm"
 			(at 168.0 160.0 0)
 			(show_name no)
@@
 		(on_board yes)
 		(in_pos_files yes)
-		(dnp no)
+		(dnp yes)
 		(property "Reference" "U1"
 			(at 55.0 110.0 0)
@@
 			)
 		)
-		(property "Description" ""
+		(property "Description" "4-pin fan header 2.54mm"
 			(at 168.0 122.0 0)
 			(show_name no)

Commit message: Fix BOM/CPL designator mismatch rejected by JLCPCB
JLCPCB meldete beidseitig fehlende Designatoren. Zwei Ursachen:

Bereichsschreibweise. Die BOM fasste Designatoren zu "R1-R4", "J2-J5",
"R9-R12" zusammen, die CPL listet sie einzeln. JLCPCB gleicht beide Dateien
designatorweise ab und kennt keine Bereiche - daher "R2,R3,R4,... don't
exist in the BOM file". collapse() schreibt jetzt vollstaendige Kommalisten.

Erfundene Designatoren fuer die Fassungen. U1-SKT1/U1-SKT2 gibt es auf der
Platine nicht: die Buchsenleisten haben kein eigenes Schaltplan-Symbol, ihre
Loecher sind die 14 Durchsteckpads des XIAO-Footprints. Ohne CPL-Eintrag
weist JLCPCB die Zeile zurueck.

Aufgeloest, indem U1 nicht mehr DNP ist und die Fassungsposition fuehrt: der
Comment beschreibt jetzt die zwei 1x7-Buchsenleisten, das Modul wird spaeter
gesteckt. Das ist die physische Wahrheit - dort sitzen Fassungen, kein
Modul. Alternativ waeren die Fassungen ganz aus der Bestueckung gefallen und
haetten 40 Stueck Handarbeit bedeutet.

DNP-Aenderung in Schaltplan und Platine, damit beide konsistent bleiben.

Geprueft: 23 Designatoren in BOM und CPL, deckungsgleich, keine Abweichung
in beide Richtungen. Alle BOM-Zeilen vierspaltig, Mehrfach-Designatoren
korrekt gequotet. DRC unveraendert.
Parts:
- U1: now fitted
Changed lines of the file:
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@@
 		(on_board yes)
 		(in_pos_files yes)
-		(dnp yes)
+		(dnp no)
 		(property "Reference" "U1"
 			(at 55.0 110.0 0)
